File: PCB/kicad/macropad.kicad_pcb (KiCad board)
At the start: 2 copper layers, 99.8 x 92 mm, 77 parts, among them J1 OLED_128x32, J2 4P4C, SW1 RESET_Push, SW2 RotaryEncoder_Switch, SW3 RotaryEncoder_Switch, SW4 RotaryEncoder_Switch, SW5 Soft_Push, SW6 Soft_Push, SW7 Soft_Push, U1 5-Way Nav, U2 NOT Gate, U3 ON/OFF

Commit message: Routed PCB
Parts:
- added H1: Pad, MountingHole:MountingHole_2.2mm_M2_Pad, F.Cu at (147.8, 56.6)
- added H2: Pad, MountingHole:MountingHole_2.2mm_M2_Pad, F.Cu at (147.8, 146.1)
- added H3: Pad, MountingHole:MountingHole_2.2mm_M2_Pad, F.Cu at (239.8, 146.1)
- added H4: Pad, MountingHole:MountingHole_2.2mm_M2_Pad, F.Cu at (240.5, 55.7)
- added H5: Pad, MountingHole:MountingHole_2.2mm_M2_Pad, F.Cu at (187.8, 56.6)
- added H6: Pad, MountingHole:MountingHole_2.2mm_M2_Pad, F.Cu at (193.8, 146.1)
- J1: moved to B.Cu
- moved U3 51.1 mm to (199.9, 55.1)
- moved D13 23.1 mm to (171.6, 119.7)
- moved D14 17.8 mm to (152.5, 126.8)
- moved C9 9.27 mm to (214.7, 119.7), turned to -90 degrees
- moved C4 9.24 mm to (157.5, 88.7), turned to -90 degrees
- moved C10 9.16 mm to (195.6, 119.6), turned to -90 degrees
- moved C12 9.12 mm to (157.5, 126.7), turned to -90 degrees
- moved C2 9.04 mm to (195.5, 81.5), turned to -90 degrees
- moved C6 9.01 mm to (195.4, 100.7), turned to -90 degrees
- moved C11 8.98 mm to (176.4, 119.7), turned to -90 degrees
- moved C7 8.97 mm to (176.5, 100.6), turned to -90 degrees
- moved C3 8.97 mm to (176.4, 81.6), turned to -90 degrees
- moved C1 8.93 mm to (214.4, 81.5), turned to -90 degrees
- moved C8 8.83 mm to (157.1, 107.8), turned to -90 degrees
- moved C5 8.70 mm to (214.1, 100.7), turned to -90 degrees
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Routing:
- net GND: track 529.4 -> 461.4 mm, vias 39 -> 14
- net +5V: track 86.9 -> 48.5 mm, vias 4 -> 1
- net Net-(J2-V): track 48.5 -> 16.5 mm
- net Net-(D12-DOUT): track 39.0 -> 14.3 mm, vias 2 -> 0
- net Net-(D1-VDD): track 286.9 -> 265.1 mm, vias 29 -> 12
- net Net-(D13-DOUT): track 37.1 -> 17.4 mm, vias 4 -> 2
- net SDA: track 88.6 -> 75.5 mm, vias 2 -> 0
- net ENC SW: track 93.7 -> 106.5 mm, vias 4 -> 3
- net B2: track 47.5 -> 56.4 mm, vias 0 -> 1
- net Net-(U2-A): track 68.4 -> 61.1 mm, vias 1 -> 0
- net ROW1: track 122.3 -> 128.4 mm, vias 2 -> 1
- net COL3: track 132.8 -> 128.1 mm, vias 1 -> 0
- net DP4T 2: track 105.7 -> 101.6 mm, vias 2 -> 3
- net COL2: track 147.4 -> 143.9 mm, vias 3 -> 0
- net DP4T 1: track 103.4 -> 100.0 mm, vias 2 -> 1
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Other:
- board size 99.8 x 92 mm -> 100 x 97.5 mm

Commit message: v2 schematic
Parts:
- removed U3: ON/OFF, SK12D07VG4:SK12D07VG4
- added C13: 0.1uf, Capacitor_SMD:C_1206_3216Metric, B.Cu at (176.2, 109.8)
- added C14: 0.1uf, Capacitor_SMD:C_1206_3216Metric, B.Cu at (157.2, 119.3)
- added C15: 0.1uf, Capacitor_SMD:C_1206_3216Metric, B.Cu at (138.1, 119.3)
- added D33: 1N4148, macropad_components:Diode_DO-35, B.Cu at (142.6, 133.3)
- added D34: 1N4148, macropad_components:Diode_DO-35, B.Cu at (123.6, 133.3)
- added D35: 1N4148, macropad_components:Diode_DO-35, B.Cu at (221.5, 105.7)
- added D36: 1N4148, macropad_components:Diode_DO-35, B.Cu at (155.4, 67.6)
- added D37: 1N4148, macropad_components:Diode_DO-35, B.Cu at (152.4, 67.6)
- added D38: 1N4148, macropad_components:Diode_DO-35, B.Cu at (149.4, 67.6)
- added MX13: KS33_SW_solder, macropad_components:SW_KS33_1u, F.Cu at (166.7, 114.3)
- added MX14: KS33_SW_solder, macropad_components:SW_KS33_1u, F.Cu at (147.6, 123.8)
- added MX15: KS33_SW_solder, macropad_components:SW_KS33_1u, F.Cu at (128.6, 123.8)
- C1, C10, C11, C12, C2, C3, C4, C5, C6, C7, C8, C9: footprint ScottoKeebs_Components:Capacitor_0603 -> Capacitor_SMD:C_1206_3216Metric
- D1, D13, D14, D2, D3, D4, D5, D6, D7, D8: footprint ScottoKeebs_Components:LED_SK6812MINI -> macropad_components:LED_SK6812MINI
- D10, D9: value LED -> LED_SK6812MINI; footprint LED_THT:LED_D1.8mm_W3.3mm_H2.4mm -> macropad_components:LED_SK6812MINI; moved to B.Cu
- D11, D12: value LED_SK6812MINI -> LED; footprint ScottoKeebs_Components:LED_SK6812MINI -> LED_THT:LED_D3.0mm; moved to F.Cu
- D15, D16, D17: value 1N4148 -> LED_SK6812MINI; footprint ScottoKeebs_Components:Diode_DO-35 -> macropad_components:LED_SK6812MINI
- D18, D20, D21, D22, D23, D25, D26, D27, D28, D30, D31, D32: footprint ScottoKeebs_Components:Diode_DO-35 -> macropad_components:Diode_DO-35
- D19: value 1N4148W -> 1N4148; footprint ScottoKeebs_Components:Diode_DO-35 -> macropad_components:Diode_DO-35
- D24, D29: value 1N4148W -> 1N4148; footprint ScottoKeebs_Components:Diode_DO-35 -> macropad_components:Diode_DO-35; moved to B.Cu
- J1: footprint B4B-XH-AM__LF__SN_:JST_B4B-XH-AM__LF__SN_ -> Connector_Wire:SolderWire-0.25sqmm_1x04_P4.2mm_D0.65mm_OD1.7mm; moved to F.Cu
- J2: footprint B4B-XH-AM__LF__SN_:JST_B4B-XH-AM__LF__SN_ -> Connector_Wire:SolderWire-0.25sqmm_1x01_D0.65mm_OD2mm; moved to F.Cu
- MX1, MX10, MX11, MX12, MX2, MX3, MX4, MX5, MX6, MX7, MX8, MX9: footprint marbastlib-xp-gateron_lp:SW_KS33_1u -> macropad_components:SW_KS33_1u
- R1, R4, R5, R6, R7: footprint Resistor_SMD:R_0603_1608Metric -> Resistor_THT:R_Axial_DIN0207_L6.3mm_D2.5mm_P10.16mm_Horizontal; moved to B.Cu
- R2: value 330Ω -> 18k; footprint Resistor_SMD:R_0603_1608Metric -> Resistor_THT:R_Axial_DIN0207_L6.3mm_D2.5mm_P10.16mm_Horizontal
- R3: value 18k -> 330Ω; footprint Resistor_SMD:R_0603_1608Metric -> Resistor_THT:R_Axial_DIN0207_L6.3mm_D2.5mm_P10.16mm_Horizontal; moved to B.Cu
- S1: moved to B.Cu
- SW1: footprint TL1105VF160Q:SW_TL1105VF160Q -> Button_Switch_SMD:SW_SPST_FSMSM; moved to F.Cu
- SW2: footprint CKW12:CKW12 -> macropad_components:CKW12
- U1: footprint MU-AS90R:MUAS90R -> macropad_components:MUAS90R
- U2: value NOT Gate -> ON/OFF; footprint SN74LVC1G14DBVRE4:SOT95P280X145-5N -> macropad_components:SK12D07VG4; moved to F.Cu
- moved H2 136.3 mm to (246.4, 52.1)
- moved H3 123.3 mm to (116.4, 146.1)
- moved H6 121.0 mm to (209.9, 26.2)
- moved D10 107.5 mm to (127.8, 99.6), turned to 180 degrees
- moved D9 91.2 mm to (146.9, 99.6), turned to 180 degrees
- moved H4 90.6 mm to (246.4, 146.1)
- moved D5 84.3 mm to (127.8, 80.6)
- moved MX5 84.2 mm to (128.6, 85.7)
- moved C5 78.4 mm to (138.1, 81.2)
- moved D12 71.9 mm to (219.2, 53.6)
- moved MX9 65.9 mm to (147.6, 104.8)
- moved MX10 65.9 mm to (128.6, 104.8)
- moved D11 61.3 mm to (219.2, 59.0)
- moved C9 60.7 mm to (157.2, 100.3)
- moved C10 60.7 mm to (138.1, 100.3)
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Connections:
- A1 pad 10: BUTTONS -> SCR A
- A1 pad 11: COL0 -> BUTTONS
- A1 pad 12: COL1 -> ROW0
- A1 pad 14: COL2 -> DP4T 2
- A1 pad 15: COL3 -> DP4T 1
- A1 pad 16: ENC SW -> COL0
- A1 pad 17: LED 1 -> COL1
- A1 pad 19: SCR A -> COL2
- A1 pad 20: SCR B -> COL4
- A1 pad 21: DP4T 1 -> A1
- A1 pad 22: DP4T 2 -> COL3
- A1 pad 25: A1 -> A2
- A1 pad 26: B1 -> B2
- A1 pad 27: A2 -> ROW1
- A1 pad 29: B2 -> ROW2
- A1 pad 32: LED 2 -> ENC SW
- A1 pad 33: GND -> unconnected-(A1-AGND-Pad33)
- A1 pad 34: unconnected-(A1-GPIO28_ADC2-Pad34) -> B1
- A1 pad 6: ROW0 -> LED 1
- A1 pad 7: ROW1 -> LED 2
- A1 pad 9: ROW2 -> SCR B
- C1 pad 1: Net-(D1-VDD) -> +5V
- C10 pad 1: Net-(D1-VDD) -> +5V
- C11 pad 1: Net-(D1-VDD) -> +5V
- C12 pad 1: Net-(D1-VDD) -> +5V
- C2 pad 1: Net-(D1-VDD) -> +5V
- C3 pad 1: Net-(D1-VDD) -> +5V
- C4 pad 1: Net-(D1-VDD) -> +5V
- C5 pad 1: Net-(D1-VDD) -> +5V
- C6 pad 1: Net-(D1-VDD) -> +5V
- C7 pad 1: Net-(D1-VDD) -> +5V
- C8 pad 1: Net-(D1-VDD) -> +5V
- C9 pad 1: Net-(D1-VDD) -> +5V
- D1 pad 1: Net-(D1-VDD) -> +5V
- D10 pad 1: GND -> +5V
- D10 pad 2: Net-(D10-A) -> Net-(D10-DOUT)
- D11 pad 1: Net-(D1-VDD) -> GND
- D11 pad 2: Net-(D11-DOUT) -> Net-(D11-A)
- D12 pad 1: Net-(D1-VDD) -> GND
- D12 pad 2: Net-(D12-DOUT) -> Net-(D12-A)
- D13 pad 1: Net-(D1-VDD) -> +5V
- D13 pad 4: Net-(D12-DOUT) -> Net-(D13-DIN)
- D14 pad 1: Net-(D1-VDD) -> +5V
- D14 pad 2: unconnected-(D14-DOUT-Pad2) -> Net-(D14-DOUT)
- D15 pad 1: ROW0 -> +5V
- D15 pad 2: Net-(D15-A) -> Net-(D15-DOUT)
- D16 pad 1: ROW0 -> +5V
- D16 pad 2: Net-(D16-A) -> Net-(D16-DOUT)
- D17 pad 1: ROW0 -> +5V
- D17 pad 2: Net-(D17-A) -> unconnected-(D17-DOUT-Pad2)
- D2 pad 1: Net-(D1-VDD) -> +5V
- D20 pad 1: ROW1 -> ROW0
- D21 pad 1: ROW1 -> ROW0
- D22 pad 1: ROW1 -> ROW0
- D23 pad 1: ROW1 -> ROW0
- D25 pad 1: ROW2 -> ROW1
- D26 pad 1: ROW2 -> ROW1
- D27 pad 1: ROW2 -> ROW1
- D28 pad 1: ROW2 -> ROW1
- D29 pad 1: ROW2 -> ROW1
- D3 pad 1: Net-(D1-VDD) -> +5V
- D30 pad 1: BUTTONS -> ROW2
- D31 pad 1: BUTTONS -> ROW2
- D32 pad 1: BUTTONS -> ROW2
- D4 pad 1: Net-(D1-VDD) -> +5V
- D4 pad 4: Net-(D3-DOUT) -> Net-(D4-DIN)
- D5 pad 1: Net-(D1-VDD) -> +5V
- D5 pad 2: Net-(D5-DOUT) -> Net-(D10-DIN)
- D6 pad 1: Net-(D1-VDD) -> +5V
- D6 pad 4: Net-(D5-DOUT) -> Net-(D3-DOUT)
- D7 pad 1: Net-(D1-VDD) -> +5V
- D8 pad 1: Net-(D1-VDD) -> +5V
- D8 pad 2: Net-(D11-DIN) -> Net-(D13-DIN)
- D9 pad 1: GND -> +5V
- D9 pad 2: Net-(D9-A) -> Net-(D4-DIN)
- J2 pad 1: USBG -> Net-(J2-Pin_1)
- MX1 pad 2: Net-(D15-A) -> Net-(D18-A)
- MX10 pad 1: COL1 -> COL4
- MX10 pad 2: Net-(D26-A) -> Net-(D28-A)
- MX11 pad 1: COL2 -> COL0
- MX11 pad 2: Net-(D27-A) -> Net-(D30-A)
- MX12 pad 1: COL3 -> COL1
- MX12 pad 2: Net-(D28-A) -> Net-(D31-A)
- MX2 pad 2: Net-(D16-A) -> Net-(D19-A)
- MX3 pad 2: Net-(D17-A) -> Net-(D20-A)
- MX4 pad 2: Net-(D18-A) -> Net-(D21-A)
- MX5 pad 1: COL0 -> COL4
- MX5 pad 2: Net-(D20-A) -> Net-(D22-A)
- MX6 pad 1: COL1 -> COL0
- MX6 pad 2: Net-(D21-A) -> Net-(D24-A)
- MX7 pad 1: COL2 -> COL1
- MX7 pad 2: Net-(D22-A) -> Net-(D25-A)
- MX8 pad 1: COL3 -> COL2
- MX8 pad 2: Net-(D23-A) -> Net-(D26-A)
- MX9 pad 1: COL0 -> COL3
- MX9 pad 2: Net-(D25-A) -> Net-(D27-A)
- R2 pad 1: BACKLIGHT -> 5-WAY NAV
- R2 pad 2: Net-(D1-DIN) -> Net-(U1-NO_2)
- R3 pad 1: 5-WAY NAV -> BACKLIGHT
- R3 pad 2: Net-(U1-NO_2) -> Net-(D1-DIN)
- R6 pad 2: Net-(D9-A) -> Net-(D11-A)
- R7 pad 2: Net-(D10-A) -> Net-(D12-A)
- S1 pad 1: Net-(U2-A) -> unconnected-(S1-Pad1)
- SW2 pad 2: Net-(D19-A) -> Net-(D23-A)
- SW3 pad S2: Net-(D24-A) -> Net-(D29-A)
- SW4 pad S2: Net-(D29-A) -> Net-(D35-A)
- SW5 pad 1: COL0 -> ROW2
- SW5 pad 2: Net-(D30-A) -> Net-(D36-A)
- SW6 pad 1: COL1 -> ROW2
- SW6 pad 2: Net-(D31-A) -> Net-(D37-A)
- SW7 pad 1: COL2 -> ROW2
- SW7 pad 2: Net-(D32-A) -> Net-(D38-A)
- U2 pad 1: (no net) -> unconnected-(U2-Pad1)
- U2 pad 2: Net-(U2-A) -> +5V
Routing:
- net GND: track 461.4 -> 0.00 mm, vias 14 -> 0
- net Net-(D1-VDD): track 265.1 -> 0.00 mm, vias 12 -> 0
- net COL2: track 143.9 -> 0.00 mm
- net ROW2: track 143.6 -> 0.00 mm, vias 3 -> 0
- net COL1: track 133.7 -> 0.00 mm, vias 1 -> 0
- net ROW1: track 128.4 -> 0.00 mm, vias 1 -> 0
- net COL3: track 128.1 -> 0.00 mm
- net COL0: track 125.1 -> 0.00 mm, vias 4 -> 0
- net ROW0: track 112.8 -> 0.00 mm
- net ENC SW: track 106.5 -> 0.00 mm, vias 3 -> 0
- net DP4T 2: track 101.6 -> 0.00 mm, vias 3 -> 0
- net DP4T 1: track 100.0 -> 0.00 mm, vias 1 -> 0
- net 5-WAY NAV: track 95.0 -> 0.00 mm, vias 1 -> 0
- net BUTTONS: track 88.3 -> 0.00 mm
- net SCL: track 79.9 -> 0.00 mm
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Other:
- board size 100 x 97.5 mm -> 138.1 x 101.8 mm

Commit message: Routed PCB v2
Parts:
- removed D38: 1N4148, macropad_components:Diode_DO-35
- removed the U1 at (232.3, 137.4)
- added R10: 10k, Resistor_THT:R_Axial_DIN0207_L6.3mm_D2.5mm_P10.16mm_Horizontal, B.Cu at (173.2, 53.3)
- added R8: 10k, Resistor_THT:R_Axial_DIN0207_L6.3mm_D2.5mm_P10.16mm_Horizontal, B.Cu at (180.4, 63.4)
- added R9: 10k, Resistor_THT:R_Axial_DIN0207_L6.3mm_D2.5mm_P10.16mm_Horizontal, B.Cu at (176.8, 63.4)
- added SW2: SW_SPST, Button_Switch_SMD:SW_DIP_SPSTx01_Slide_6.7x4.1mm_W6.73mm_P2.54mm_LowProfile_JPin, F.Cu at (231.7, 57.0)
- D1, D2: value LED_SK6812MINI -> LED; footprint macropad_components:LED_SK6812MINI -> LED_THT:LED_D3.0mm
- D11, D12: value LED -> LED_SK6812MINI; footprint LED_THT:LED_D3.0mm -> macropad_components:LED_SK6812MINI; moved to B.Cu
- H1, H2, H3, H4, H5, H6: moved to B.Cu
- J1: footprint Connector_Wire:SolderWire-0.25sqmm_1x04_P4.2mm_D0.65mm_OD1.7mm -> Connector_PinHeader_2.54mm:PinHeader_1x04_P2.54mm_Vertical
- J2: value 4P4C -> 01x01_Pin; moved to B.Cu
- R1: value 12k -> 330
- R2: value 18k -> 330
- R3: value 330Ω -> 12k
- R4: value 5.1k -> 18k
- R5: value 33k -> 5.1k
- R6: value 330Ω -> 33k
- R7: value 330 -> 330Ω
- S1: value DP4T Slide Switch -> PCM13SMTR; footprint Connector_PinHeader_2.54mm:PinHeader_2x06_P2.54mm_Vertical -> macropad_components:SW_PCM13SMTR; moved to F.Cu
- SW3: renamed from SW2; value RotaryEncoder_Switch -> ScrollEncoder_Switch
- SW6: renamed from SW5; value Soft_Push -> SW_Push; footprint Button_Switch_THT:SW_PUSH_6mm -> Button_Switch_THT:SW_PUSH_6mm_H4.3mm
- SW7: renamed from SW6; value Soft_Push -> SW_Push; footprint Button_Switch_THT:SW_PUSH_6mm -> Button_Switch_THT:SW_PUSH_6mm_H4.3mm
- SW8: renamed from SW7; value Soft_Push -> SW_Push; footprint Button_Switch_THT:SW_PUSH_6mm -> Button_Switch_THT:SW_PUSH_6mm_H4.3mm
- U1: renamed from U2; value ON/OFF -> 5-Way Nav; footprint macropad_components:SK12D07VG4 -> macropad_components:MUAS90R
- moved D34 119.0 mm to (241.1, 114.7), turned to -90 degrees
- moved D12 102.3 mm to (127.8, 99.6), turned to 0 degrees
- moved R2 95.2 mm to (184.0, 53.3), turned to -90 degrees
- moved D33 86.0 mm to (191.7, 62.7), turned to 90 degrees
- moved R1 85.8 mm to (187.5, 63.4)
- moved D11 82.9 mm to (146.9, 99.6), turned to 0 degrees
- moved R6 81.9 mm to (210.7, 142.0)
- moved D28 76.8 mm to (199.8, 123.8)
- moved U1 76.6 mm to (232.3, 136.9)
- moved D7 57.9 mm to (127.8, 80.6)
- moved D6 57.9 mm to (146.9, 80.6)
- moved R3 56.4 mm to (221.5, 142.0)
- moved R7 49.7 mm to (219.1, 98.5)
- moved D23 42.6 mm to (199.8, 104.8)
- moved D29 41.6 mm to (180.7, 123.8), turned to 0 degrees
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- renumbered SW3 to SW4, SW4 to SW5
Connections:
- net Net-(D35-A) renamed /Switch Matrix/2S2
- A1 pad 10: SCR A -> ROW0
- A1 pad 11: BUTTONS -> ROW1
- A1 pad 12: ROW0 -> ROW2
- A1 pad 14: DP4T 2 -> ROW3
- A1 pad 15: DP4T 1 -> COL0
- A1 pad 16: COL0 -> COL1
- A1 pad 17: COL1 -> COL2
- A1 pad 19: COL2 -> COL3
- A1 pad 22: COL3 -> A2
- A1 pad 25: A2 -> B1
- A1 pad 27: ROW1 -> LED 1
- A1 pad 29: ROW2 -> LED 2
- A1 pad 32: ENC SW -> SP3T
- A1 pad 34: B1 -> unconnected-(A1-GPIO28_ADC2-Pad34)
- A1 pad 6: LED 1 -> SCR A
- A1 pad 7: LED 2 -> SCR B
- A1 pad 9: SCR B -> S0
- D1 pad 1: +5V -> GND
- D1 pad 2: Net-(D1-DOUT) -> Net-(D1-A)
- D11 pad 1: GND -> +5V
- D11 pad 2: Net-(D11-A) -> Net-(D11-DOUT)
- D12 pad 1: GND -> +5V
- D12 pad 2: Net-(D12-A) -> Net-(D12-DOUT)
- D13 pad 4: Net-(D13-DIN) -> Net-(D10-DOUT)
- D16 pad 2: Net-(D16-DOUT) -> Net-(D11-DIN)
- D17 pad 4: Net-(D10-DOUT) -> Net-(D12-DOUT)
- D2 pad 1: +5V -> GND
- D2 pad 2: Net-(D2-DOUT) -> Net-(D2-A)
- D23 pad 1: ROW0 -> ROW1
- D28 pad 1: ROW1 -> ROW2
- D29 pad 1: ROW1 -> ROW2
- D3 pad 4: Net-(D2-DOUT) -> Net-(D3-DIN)
- D33 pad 1: ROW2 -> ROW3
- D33 pad 2: Net-(D33-A) -> /Switch Matrix/SCR2
- D34 pad 1: ROW2 -> ROW3
- D34 pad 2: Net-(D34-A) -> /Switch Matrix/1S2
- D35 pad 1: ROW2 -> ROW3
- D36 pad 1: BUTTONS -> ROW3
- D37 pad 1: BUTTONS -> ROW3
- D4 pad 4: Net-(D4-DIN) -> Net-(D3-DOUT)
- D5 pad 2: Net-(D10-DIN) -> Net-(D5-DOUT)
- D6 pad 4: Net-(D3-DOUT) -> Net-(D11-DOUT)
- D7 pad 2: Net-(D7-DOUT) -> Net-(D12-DIN)
- D8 pad 2: Net-(D13-DIN) -> Net-(D8-DOUT)
- D8 pad 4: Net-(D7-DOUT) -> Net-(D5-DOUT)
- D9 pad 2: Net-(D4-DIN) -> Net-(D10-DIN)
- D9 pad 4: Net-(D16-DOUT) -> Net-(D8-DOUT)
- H1 pad 1: unconnected-(H1-Pad1) -> GND
- H2 pad 1: unconnected-(H2-Pad1) -> GND
- H3 pad 1: unconnected-(H3-Pad1) -> GND
- H4 pad 1: unconnected-(H4-Pad1) -> GND
- H5 pad 1: unconnected-(H5-Pad1) -> GND
- H6 pad 1: unconnected-(H6-Pad1) -> GND
- MX10 pad 2: Net-(D28-A) -> Net-(D27-A)
- MX11 pad 2: Net-(D30-A) -> Net-(D28-A)
- MX12 pad 2: Net-(D31-A) -> Net-(D29-A)
- MX13 pad 2: Net-(D32-A) -> Net-(D30-A)
- MX14 pad 2: Net-(D33-A) -> Net-(D31-A)
- MX15 pad 2: Net-(D34-A) -> Net-(D32-A)
- MX6 pad 2: Net-(D24-A) -> Net-(D23-A)
- MX7 pad 2: Net-(D25-A) -> Net-(D24-A)
- MX8 pad 2: Net-(D26-A) -> Net-(D25-A)
- MX9 pad 2: Net-(D27-A) -> Net-(D26-A)
- R1 pad 1: 5-WAY NAV -> LED 1
- R1 pad 2: Net-(U1-NO_1) -> Net-(D1-A)
- R2 pad 1: 5-WAY NAV -> LED 2
- R2 pad 2: Net-(U1-NO_2) -> Net-(D2-A)
- R3 pad 1: BACKLIGHT -> 5-WAY NAV
- R3 pad 2: Net-(D1-DIN) -> Net-(U1-NO_1)
- R4 pad 2: Net-(U1-NO_4) -> Net-(U1-NO_2)
- R5 pad 2: Net-(U1-CENTER) -> Net-(U1-NO_4)
- R6 pad 1: LED 1 -> 5-WAY NAV
- R6 pad 2: Net-(D11-A) -> Net-(U1-CENTER)
- R7 pad 1: LED 2 -> BACKLIGHT
- R7 pad 2: Net-(D12-A) -> Net-(D3-DIN)
- S1 pad 1: unconnected-(S1-Pad1) -> Net-(R8-Pad2)
- S1 pad 2: unconnected-(S1-Pad2) -> Net-(R9-Pad2)
- S1 pad 3: GND -> SP3T
- S1 pad 4: DP4T 1 -> GND
- SW4 pad MP: (no net) -> GND
- SW4 pad S1: ENC SW -> COL1
- SW4 pad S2: Net-(D29-A) -> /Switch Matrix/1S2
- SW5 pad MP: (no net) -> GND
- SW5 pad S1: ENC SW -> COL2
- SW6 pad 1: ROW2 -> COL3
- SW7 pad 1: ROW2 -> COL4
- SW8 pad 1: ROW2 -> Net-(R10-Pad2)
- SW8 pad 2: Net-(D38-A) -> GND
Routing:
- net +5V: track 0.00 -> 360.3 mm, vias 0 -> 10
- net COL4: track 0.00 -> 211.9 mm, vias 0 -> 3
- net COL3: track 0.00 -> 193.5 mm, vias 0 -> 3
- net ROW2: track 0.00 -> 183.6 mm, vias 0 -> 2
- net ROW1: track 0.00 -> 158.4 mm, vias 0 -> 3
- net ROW3: track 0.00 -> 147.2 mm, vias 0 -> 4
- net COL2: track 0.00 -> 141.1 mm, vias 0 -> 1
- net ROW0: track 0.00 -> 140.3 mm, vias 0 -> 3
- net SCL: track 0.00 -> 123.6 mm, vias 0 -> 2
- net COL0: track 0.00 -> 108.0 mm, vias 0 -> 1
- net SP3T: track 0.00 -> 107.9 mm, vias 0 -> 1
- net COL1: track 0.00 -> 103.5 mm, vias 0 -> 2
- net +3.3V: track 0.00 -> 103.2 mm
- net 5-WAY NAV: track 0.00 -> 96.4 mm, vias 0 -> 1
- net S0: track 0.00 -> 92.6 mm, vias 0 -> 1
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